Commit message: update files

File: urdf/mycobot_280_m5.urdf (robot description, URDF)
Before this commit: robot mycobot_ai_no, 8 links, 7 joints
Joints:
- joint joint2: limit lower=-3.14 upper=3.14159 effort=1000.0 velocity=0.1 -> lower=-3.14 upper=3.14159 effort=1000.0 velocity=1.0
- joint joint3: limit lower=-3.14 upper=3.14159 effort=1000.0 velocity=0.1 -> lower=-3.14 upper=3.14159 effort=1000.0 velocity=1.0
- joint joint4: limit lower=-3.14 upper=3.14159 effort=1000.0 velocity=0.1 -> lower=-3.14 upper=3.14159 effort=1000.0 velocity=1.0
- joint joint5: limit lower=-3.14 upper=3.14159 effort=1000.0 velocity=0.1 -> lower=-3.14 upper=3.14159 effort=1000.0 velocity=1.0
- joint joint6: limit lower=-3.14 upper=3.14159 effort=1000.0 velocity=0.1 -> lower=-3.14 upper=3.14159 effort=1000.0 velocity=1.0
